Commit message: progressie???? idk???? wa is ros man

File: webots_ros2_turtlebot/install/webots_ros2_turtlebot/share/webots_ros2_turtlebot/resource/turtlebot_webots.urdf (robot description, URDF)
Before this commit: robot TurtleBot3 Burger Webots, 0 links, 0 joints
Links:
- added link base_footprint
- added link base_link, mass 1.0; collision box size=0.140 0.140 0.143; visual box size=0.140 0.140 0.143
- added link base_scan; visual cylinder length=0.03 radius=0.03
- added link caster_back_link; collision box size=0.030 0.009 0.020
- added link wheel_left_link, mass 0.1; collision cylinder length=0.018 radius=0.033; visual cylinder length=0.018 radius=0.033
- added link wheel_right_link, mass 0.1; collision cylinder length=0.018 radius=0.033; visual cylinder length=0.018 radius=0.033
Joints:
- added joint base_joint: type fixed, parent base_link, child base_footprint, origin xyz=0 0 0 rpy=0 0 0
- added joint caster_back_joint: type fixed, parent base_link, child caster_back_link, origin xyz=-0.081 0 -0.004 rpy=0 0 0
- added joint scan_joint: type fixed, parent base_link, child base_scan, origin xyz=0 0 0.08 rpy=0 0 0
- added joint wheel_left_joint: type continuous, parent base_link, child wheel_left_link, origin xyz=0.0 0.08 0.023 rpy=0 0 0, axis 0 1 0
- added joint wheel_right_joint: type continuous, parent base_link, child wheel_right_link, origin xyz=0.0 -0.08 0.023 rpy=0 0 0, axis 0 1 0

Commit message: whodee kheb iets gedaan en twas vooruitgang denk

File: webots_ros2_turtlebot/install/webots_ros2_turtlebot/share/webots_ros2_turtlebot/resource/turtlebot_webots.urdf (robot description, URDF)
Before this commit: robot TurtleBot3Burger, 6 links, 5 joints
Links:
- removed link base_footprint
- removed link base_link
- removed link base_scan
- removed link caster_back_link
- removed link wheel_left_link
- removed link wheel_right_link
Joints:
- removed joint base_joint
- removed joint caster_back_joint
- removed joint scan_joint
- removed joint wheel_left_joint
- removed joint wheel_right_joint
